File: combat-pcb/combat-pcb.kicad_pcb (KiCad board)
At the start: 2 copper layers, 73.4 x 41.9 mm, 22 parts, among them IC1 LSM6DSRTR, IC2 RP2, IC3 H3LIS331DLTR, J1 TSW-106-08-T-T-RA, J7 Screw_Terminal_01x02, J8 Conn_01x16_Socket, U2 AP63205WU

Commit message: placed JLCPCB order.  these are the files I sent
Routing:
- net GND: track 26.3 -> 23.8 mm
- net /SPI_COPI: track 81.6 -> 83.1 mm, vias 5 -> 4
Changed lines of the file:
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@@
 	)
 	(segment
-		(start 148.3305 99.4595)
-		(end 147.841 99.949)
-		(width 0.508)
-		(layer "F.Cu")
-		(net 6)
-	)
-	(segment
 		(start 205.664699 109.7917)
 		(end 206.108756 109.7917)
@@
 	)
 	(segment
-		(start 148.3305 97.597)
-		(end 148.3305 99.4595)
-		(width 0.508)
-		(layer "F.Cu")
-		(net 6)
-	)
-	(segment
 		(start 205.664699 109.7917)
 		(end 203.3003 109.7917)
@@
 	)
 	(segment
-		(start 208.788 106.553)
-		(end 208.407 106.172)
-		(width 0.1524)
+		(start 212.344 109.22)
+		(end 211.455 108.331)
+		(width 0.2)
 		(layer "F.Cu")
 		(net 8)
 	)
 	(segment
-		(start 208.136998 111.76)
-		(end 207.374998 110.998)
-		(width 0.1524)
+		(start 207.899 111.887)
+		(end 211.455 111.887)
+		(width 0.2)
+		(layer "F.Cu")
+		(net 8)
+	)
+	(segment
+		(start 211.455 108.331)
+		(end 211.455 108.204)
+		(width 0.2)
+		(layer "F.Cu")
+		(net 8)
+	)
+	(segment
+		(start 207.772 111.76)
+		(end 207.899 111.887)
+		(width 0.2)
 		(layer "F.Cu")
 		(net 8)
@@
 	)
 	(segment
-		(start 205.486 107.569)
-		(end 208.407 104.648)
+		(start 212.344 110.998)
+		(end 212.344 109.22)
 		(width 0.2)
 		(layer "F.Cu")
@@
 	)
 	(segment
-		(start 181.412286 110.579926)
-		(end 179.3494 110.579926)
+		(start 211.455 111.887)
+		(end 212.344 110.998)
 		(width 0.2)
 		(layer "F.Cu")
@@
 	)
 	(segment
-		(start 211.328 109.093)
-		(end 211.328 109.601)
-		(width 0.1524)
+		(start 205.486 107.569)
+		(end 208.407 104.648)
+		(width 0.2)
 		(layer "F.Cu")
 		(net 8)
 	)
 	(segment
-		(start 209.169 111.76)
-		(end 208.136998 111.76)
-		(width 0.1524)
+		(start 181.412286 110.579926)
+		(end 179.3494 110.579926)
+		(width 0.2)
 		(layer "F.Cu")
 		(net 8)
@@
 	)
 	(segment
-		(start 208.407 106.172)
-		(end 208.407 102.489)
-		(width 0.1524)
+		(start 207.374998 111.362998)
+		(end 207.772 111.76)
+		(width 0.2)
 		(layer "F.Cu")
 		(net 8)
 	)
 	(segment
-		(start 211.328 109.601)
-		(end 209.169 111.76)
-		(width 0.1524)
+		(start 207.374998 110.998)
+		(end 207.374998 111.362998)
+		(width 0.2)
 		(layer "F.Cu")
 		(net 8)
@@
 	)
 	(via
-		(at 211.328 109.093)
-		(size 0.6)
-		(drill 0.3)
-		(layers "F.Cu" "B.Cu")
-		(net 8)
-	)
-	(via
-		(at 208.788 106.553)
-		(size 0.6)
+		(at 211.455 108.204)
+		(size 0.5)
 		(drill 0.3)
 		(layers "F.Cu" "B.Cu")
@@
 	)
 	(segment
-		(start 197.398471 108.331)
-		(end 200.792471 111.725)
+		(start 183.642 108.331)
+		(end 197.398471 108.331)
 		(width 0.2)
 		(layer "B.Cu")
@@
 	)
 	(segment
-		(start 182.318106 109.674106)
-		(end 182.318106 109.654894)
+		(start 204.597 108.458)
+		(end 205.486 107.569)
 		(width 0.2)
 		(layer "B.Cu")
@@
 	)
 	(segment
-		(start 205.486 109.474)
+		(start 210.82 107.569)
 		(end 205.486 107.569)
 		(width 0.2)
@@
 	)
 	(segment
-		(start 209.296 106.553)
-		(end 211.328 108.585)
-		(width 0.1524)
+		(start 208.407 76.581)
+		(end 205.359 73.533)
+		(width 0.2)
 		(layer "B.Cu")
 		(net 8)
 	)
 	(segment
-		(start 208.788 106.553)
-		(end 209.296 106.553)
-		(width 0.1524)
+		(start 200.792471 111.725)
+		(end 203.235 111.725)
+		(width 0.2)
 		(layer "B.Cu")
 		(net 8)
 	)
 	(segment
-		(start 203.235 111.725)
-		(end 205.486 109.474)
+		(start 197.398471 108.331)
+		(end 200.792471 111.725)
 		(width 0.2)
 		(layer "B.Cu")
@@
 	)
 	(segment
-		(start 208.407 76.581)
-		(end 205.359 73.533)
+		(start 203.235 111.725)
+		(end 204.597 110.363)
 		(width 0.2)
 		(layer "B.Cu")
@@
 	)
 	(segment
-		(start 183.642 108.331)
-		(end 197.398471 108.331)
+		(start 182.318106 109.674106)
+		(end 182.318106 109.654894)
 		(width 0.2)
 		(layer "B.Cu")
@@
 	)
 	(segment
-		(start 211.328 108.585)
-		(end 211.328 109.093)
-		(width 0.1524)
+		(start 182.318106 109.654894)
+		(end 183.642 108.331)
+		(width 0.2)
 		(layer "B.Cu")
 		(net 8)
 	)
 	(segment
-		(start 200.792471 111.725)
-		(end 203.235 111.725)
+		(start 204.597 110.363)
+		(end 204.597 108.458)
 		(width 0.2)
 		(layer "B.Cu")
@@
 	)
 	(segment
-		(start 182.318106 109.654894)
-		(end 183.642 108.331)
+		(start 211.455 108.204)
+		(end 210.82 107.569)
 		(width 0.2)
 		(layer "B.Cu")
@@
 		(start 156.313 95.655)
 		(end 174.371 77.597)
-		(width 0.508)
+		(width 1.016)
 		(layer "F.Cu")
 		(net 17)
@@
 		(start 145.923 100.317)
 		(end 146.291 99.949)
-		(width 1.27)
+		(width 0.635)
 		(layer "F.Cu")
 		(net 19)
@@
 		(start 146.0555 99.7135)
 		(end 146.291 99.949)
-		(width 1.27)
+		(width 0.635)
 		(layer "F.Cu")
 		(net 19)
@@
 		(start 145.923 104.982)
 		(end 145.923 100.317)
-		(width 1.27)
+		(width 0.635)
 		(layer "F.Cu")
 		(net 19)
@@
 		(start 146.0555 97.597)
 		(end 146.0555 99.7135)
-		(width 1.27)
+		(width 0.635)
 		(layer "F.Cu")
 		(net 19)
@@
 		(start 146.0555 97.597)
 		(end 146.0555 96.705)
-		(width 1)
+		(width 0.635)
 		(layer "F.Cu")
 		(net 19)
