File: combat-pcb/combat-pcb.kicad_sch (KiCad schematic)
At the start: 17 parts, among them IC1 LSM6DSRTR, IC2 RP2, IC3 H3LIS331DLTR, J1 TSW-106-08-T-T-RA, J7 Screw_Terminal_01x02, J8 Conn_01x16_Socket, U2 AP63205WU

Commit message: placed JLCPCB order.  these are the files I sent
Changed lines of the file:
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@@
 		(on_board yes)
 		(dnp no)
-		(fields_autoplaced yes)
 		(property "Reference" "#PWR0103"
 			(at 215.9 151.13 0)
@@
 		)
 		(property "Value" "+5V"
-			(at 215.9 142.24 0)
+			(at 215.392 144.272 0)
 			(effects
 				(font
@@
 		(on_board yes)
 		(dnp no)
-		(fields_autoplaced yes)
 		(property "Reference" "#PWR032"
 			(at 220.98 133.35 0)
@@
 		)
 		(property "Value" "GND"
-			(at 220.98 132.08 0)
+			(at 221.488 125.222 0)
 			(effects
 				(font
@@
 		(on_board yes)
 		(dnp no)
-		(fields_autoplaced yes)
 		(property "Reference" "#PWR0104"
 			(at 220.98 151.13 0)
@@
 		)
 		(property "Value" "GND"
-			(at 220.98 149.86 0)
+			(at 220.98 143.002 0)
 			(effects
 				(font
@@
 		(on_board yes)
 		(dnp no)
-		(fields_autoplaced yes)
 		(property "Reference" "#PWR025"
 			(at 165.1 138.43 0)
@@
 		)
 		(property "Value" "GND"
-			(at 165.1 137.16 0)
-			(effects
-				(font
+			(at 167.64 130.81 0)
+			(effects
+				(font
